File: pcbs/corne-chocolate/hotswap/corne-chocolate.kicad_pcb (KiCad board)
At the start: 2 copper layers, 277.2 x 107.5 mm, 178 parts, among them J1 TYPE-C-31-M-13C, J2 PJ-606-6A, J3 Conn_01x04, J4 Conn_01x03, SW1 SW_Push, SW10 SW_Push, SW11 SW_Push, SW12 SW_Push, SW13 SW_Push, SW14 SW_Push, SW15 SW_Push, SW16 SW_Push, SW17 SW_Push, SW18 SW_Push, SW19 SW_Push, SW2 SW_Push, SW20 SW_Push, SW21 SW_Push, SW3 SW_Push, SW4 SW_Push, SW5 SW_Push, SW6 SW_Push, SW7 SW_Push, SW8 SW_Push, SW9 SW_Push, U1 RP2040, U2 NCP1117LPST33T3G, U3 TPD4E05U06DQAR, U4 W25Q128JVSIQ, Y1 12MHz 18pF

Commit message: Moved VIAs in compliance with JLCPCB engineers
Parts:
- moved C4 0.23 mm to (132.3, 133.1)
- moved C9 0.19 mm to (139.5, 142.2)
Routing:
- net GNDR: track 98.6 -> 157.8 mm
- net GND: track 123.0 -> 181.0 mm
- net +5V: track 117.5 -> 105.8 mm
- net Net-(R6-Pad2): track 8.85 -> 12.2 mm
- net Net-(rJP1-A): track 58.6 -> 61.6 mm
- net Net-(U1-RUN): track 22.2 -> 25.0 mm
- net Net-(rLED15-DOUT): track 35.4 -> 38.0 mm
- net Net-(rLED8-DOUT): track 33.4 -> 35.8 mm
- net Net-(rLED4-DOUT): track 33.0 -> 35.3 mm
- net Net-(JP1-A): track 27.5 -> 25.6 mm
- net /right/TX: track 98.8 -> 96.9 mm
- net Net-(D1-K): track 527.1 -> 528.9 mm
- net Net-(EXLED1-DIN): track 197.3 -> 199.2 mm
- net Net-(rD1-K): track 567.6 -> 565.8 mm
- net Net-(rLED12-DOUT): track 33.4 -> 35.1 mm
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Other:
- rule pad_to_mask_clearance: 0.2 -> 0
- board text added: "Modified by Fredrik L 2024-04"
